File: board_neo.kicad_sch (KiCad schematic)
At the start: 7 parts, among them J1 Conn_01x07, J2 Conn_02x02_Odd_Even, J5 DE9_Receptacle

Commit message: Finalize design
Parts:
- removed J5: DE9_Receptacle, symbol Connector:DE9_Receptacle
- removed e: Conn_01x11, symbol Connector_Generic:Conn_01x11
- added C1, C3, C4, C5: 1nF, Capacitor_SMD:C_0805_2012Metric_Pad1.18x1.45mm_HandSolder, symbol Device:C_Small
- added C2: C_Polarized_Small, Capacitor_THT:CP_Radial_D5.0mm_P2.50mm, symbol Device:C_Polarized_Small
- added D1: SP7538P, Package_DFN_QFN:UDFN-9_1.0x3.8mm_P0.5mm, symbol Power_Protection:SP7538P
- added D2: D_Small, Diode_SMD:D_SOD-123, symbol Device:D_Small
- added H1, H2, H3, H4: MountingHole_Pad, MountingHole:MountingHole_3.2mm_M3_ISO7380_Pad, symbol Mechanical:MountingHole_Pad
- added J3: DE9_Receptacle_MountingHoles, Connector_Dsub:DSUB-9_Female_Vertical_P2.77x2.84mm_MountingHoles, symbol Connector:DE9_Receptacle_MountingHoles
- added J4: Conn_01x12, Connector_PinHeader_2.54mm:PinHeader_1x12_P2.54mm_Vertical, symbol Connector_Generic:Conn_01x12
- added R3, R5, R6, R7: 470R, Resistor_SMD:R_0603_1608Metric_Pad0.98x0.95mm_HandSolder, symbol Device:R_Small
- added RV1: R_Potentiometer_Small, Potentiometer_THT:Potentiometer_Bourns_3386F_Vertical, symbol Device:R_Potentiometer_Small
- added U1: ~, fsaev_lib:LM2596_DCDC_dboard, symbol fsaev_lib:LM2596_DCDC_dboard
- J1: footprint (none) -> Connector_PinHeader_2.54mm:PinHeader_1x07_P2.54mm_Vertical
- J2: footprint (none) -> Connector_Molex:Molex_Nano-Fit_105310-xx04_2x02_P2.50mm_Vertical
- R1, R2: footprint (none) -> Resistor_SMD:R_0603_1608Metric_Pad0.98x0.95mm_HandSolder
Connections:
- net Earth: now also C1.2, C2.2, C3.2, C4.2, C5.2, D1.3 (A), D2.2 (A), H1.1, H2.1, H3.1, H4.1, J3.0 (PAD), J3.3, J3.4, J3.5, J4.12 (Pin_12), J4.2 (Pin_2), RV1.3, U1.1 (mthole_pad1), U1.2 (mthole_pad2), U1.4 (in-), U1.6 (out-)
- net VIN: now also C2.1, D2.1 (K), J3.8, J3.9, U1.3 (in+)
- net at A1.11 (D8): now also J4.3 (Pin_3)
- net at A1.10 (D7): now also J4.4 (Pin_4)
- net at A1.9 (D6): now also J4.5 (Pin_5)
- net at A1.8 (D5): now also J4.6 (Pin_6)
- net at A1.7 (D4): now also J4.7 (Pin_7)
- net at A1.6 (D3): now also J4.8 (Pin_8)
- net at A1.5 (D2): now also J4.9 (Pin_9)
- net at A1.14 (D11): now also R7.2
- net at A1.15 (D12): now also R6.2
- net at A1.16 (D13): now also R5.2
- net at A1.19 (A0): now also R3.2
- new net: C5.1, D1.1 (K1), J3.7, R7.1
- new net: C3.1, D1.4 (K3), J3.6, R5.1
- new net: J4.10 (Pin_10), RV1.2
- new net: C4.1, D1.2 (K2), J3.2, R6.1
- new net: C1.1, D1.5 (K4), J3.1, R3.1
- new net VBUCK: J4.1 (Pin_1), J4.11 (Pin_11), RV1.1, U1.5 (out+)
Other:
- note added: "470R/1nF : 0.338 MHz cutoff"
- moved on the sheet: J2, R1, R2
